File: PCB/viagrid/viagrid.kicad_sch (KiCad schematic)
At the start: 1 part

Commit message: cleans up a bunch of stuff
Parts:
- removed R1: R, Resistor_SMD:R_0201_0603Metric, symbol Device:R
- added TP1: TestPoint, TestPoint:TestPoint_Pad_1.0x1.0mm, symbol Connector:TestPoint
Connections:
- net GND: now also TP1.1
Changed lines of the file:
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@@
 	(paper "A4")
 	(symbol
-		(lib_id "Device:R")
-		(at 85.725 57.785 0)
+		(lib_id "Connector:TestPoint")
+		(at 106.68 81.28 270)
 		(unit 1)
 		(exclude_from_sim no)
@@
 		(dnp no)
 		(fields_autoplaced yes)
-		(property "Reference" "R1"
-			(at 87.503 56.525 0)
+		(property "Reference" "TP1"
+			(at 111.379 80.02 90)
 			(effects
 				(font
@@
 			)
 		)
-		(property "Value" "R"
-			(at 87.503 59.045 0)
+		(property "Value" "TestPoint"
+			(at 111.379 82.54 90)
 			(effects
 				(font
@@
 			)
 		)
-		(property "Footprint" "Resistor_SMD:R_0201_0603Metric"
-			(at 83.947 57.785 90)
+		(property "Footprint" "TestPoint:TestPoint_Pad_1.0x1.0mm"
+			(at 106.68 86.36 0)
 			(effects
 				(font
@@
 		)
 		(property "Datasheet" "~"
-			(at 85.725 57.785 0)
+			(at 106.68 86.36 0)
 			(effects
 				(font
@@
 			)
 		)
-		(property "Description" "Resistor"
-			(at 85.725 57.785 0)
+		(property "Description" "test point"
+			(at 106.68 81.28 0)
 			(effects
 				(font
@@
 		(pin "1"
 		)
-		(pin "2"
-		)
 		(instances
 			(project ""
 				(path "/efce478c-7ae4-454c-9230-ffcb4459a9b8"
-					(reference "R1")
+					(reference "TP1")
 					(unit 1)
 				)
@@
 	(symbol
 		(lib_id "power:GND")
-		(at 85.725 61.595 0)
+		(at 106.68 81.28 270)
 		(unit 1)
 		(exclude_from_sim no)
@@
 		(fields_autoplaced yes)
 		(property "Reference" "#PWR01"
-			(at 85.725 67.945 0)
+			(at 100.33 81.28 0)
 			(effects
 				(font
@@
 		)
 		(property "Value" "GND"
-			(at 85.725 65.776 0)
+			(at 103.5051 81.28 90)
 			(effects
 				(font
 					(size 1.27 1.27)
 				)
+				(justify right)
 			)
 		)
 		(property "Footprint" ""
-			(at 85.725 61.595 0)
+			(at 106.68 81.28 0)
 			(effects
 				(font
@@
 		)
 		(property "Datasheet" ""
-			(at 85.725 61.595 0)
+			(at 106.68 81.28 0)
 			(effects
 				(font
@@
 		)
 		(property "Description" "Power symbol creates a global label with name \"GND\" , ground"
-			(at 85.725 61.595 0)
+			(at 106.68 81.28 0)
 			(effects
 				(font
