File: test/blade-programmer/blade-programmer.kicad_sch (KiCad schematic)
At the start: 45 parts, among them J1 SWD_10, J2 display, J3 STYLUS, J4 SW1, J5 Barrel_Jack_MountingPin, J6 SW2, U1 STM32F031C6Tx, U4 AP1117-33, U5 MC34063AD, Y1 8MHz

Commit message: cleans up a bunch of stuff
Other:
- moved on the sheet: C6, D9, J3, R14
